Commit message: added wheels and joints

File: catkin_ws/src/my_robot/urdf/my_robot.xacro (robot description, xacro)
@@ -55,3 +55,65 @@
     </visual>
   </link>
+  <link name="left_wheel">
+    <collision>
+        <origin xyz="0 0 0" rpy="0 1.507 1.507"/>
+        <geometry>
+            <cylinder radius="0.1" length="0.05"/>
+        </geometry>
+    </collision>
+    <inertial>
+        <origin xyz="0 0 0" rpy="0 1.507 1.507"/>
+        <mass value="5.0"/>
+        <inertia
+            ixx="0.1" ixy="0" ixz="0"
+            iyy="0.1" iyz="0"
+            izz="0.1"
+        />
+    </inertial>
+    <visual>
+        <origin xyz="0 0 0" rpy="0 1.507 1.507"/>
+        <geometry>
+            <cylinder radius="0.1" length="0.05"/>
+        </geometry>
+    </visual>
+  </link>
+  <link name="right_wheel">
+    <collision>
+        <origin xyz="0 0 0" rpy="0 1.507 1.507"/>
+        <geometry>
+            <cylinder radius="0.1" length="0.05"/>
+        </geometry>
+    </collision>
+    <inertial>
+        <origin xyz="0 0 0" rpy="0 1.507 1.507"/>
+        <mass value="5.0"/>
+        <inertia
+            ixx="0.1" ixy="0" ixz="0"
+            iyy="0.1" iyz="0"
+            izz="0.1"
+        />
+    </inertial>
+    <visual>
+        <origin xyz="0 0 0" rpy="0 1.507 1.507"/>
+        <geometry>
+            <cylinder radius="0.1" length="0.05"/>
+        </geometry>
+    </visual>
+  </link> -->
+  <joint type="continuous" name="left_wheel_hinge">
+    <origin xyz="0 0.15 0" rpy="0 0 0"/>
+    <child link="left_wheel"/>
+    <parent link="chassis"/>
+    <axis xyz="0 1 0" rpy="0 0 0"/>
+    <limit effort="10000" velocity="1000"/>
+    <dynamics damping="1.0" friction="1.0"/>
+  </joint>
+  <joint type="continuous" name="right_wheel_hinge">
+    <origin xyz="0 -0.15 0" rpy="0 0 0"/>
+    <child link="right_wheel"/>
+    <parent link="chassis"/>
+    <axis xyz="0 1 0" rpy="0 0 0"/>
+    <limit effort="10000" velocity="1000"/>
+    <dynamics damping="1.0" friction="1.0"/>
+  </joint>
 </robot>

Commit message: added camera and lidar(with mesh)

File: catkin_ws/src/my_robot/urdf/my_robot.xacro (robot description, xacro)
@@ -117,3 +117,58 @@
     <dynamics damping="1.0" friction="1.0"/>
   </joint>
+  <link name="camera">
+    <origin xyz="0 0 0" rpy="0 0 0"/>
+    <collision>
+        <geometry>
+            <box size="0.05 0.05 0.05"/>
+        </geometry>
+    </collision>
+    <inertial>
+        <mass value="0.1"/>
+        <box_inertia m="0.1" x="0.05" y="0.05" z="0.05"/>
+        <inertia
+            ixx="1e-6" ixy="0" ixz="0"
+            iyy="1e-6" iyz="0"
+            izz="1e-6"
+        />
+    </inertial>
+    <visual>
+        <geometry>
+            <box size="0.05 0.05 0.05"/>
+        </geometry>
+    </visual>
+  </link>
+  <joint type="fixed" name="camera_joint">
+    <origin xyz="0.2 0 0" rpy="0 0 0"/>
+    <child link="camera"/>
+    <parent link="chassis"/>
+    <axis xyz="0 1 0"/>
+  </joint>
+  <link name="hokuyo">
+    <origin xyz="0 0 0" rpy="0 0 0"/>
+    <collision>
+        <geometry>
+            <box size="0.1 0.1 0.1"/>
+        </geometry>
+    </collision>
+    <inertial>
+        <mass value="1e-5"/>
+        <inertia
+            ixx="1e-6" ixy="0" ixz="0"
+            iyy="1e-6" iyz="0"
+            izz="1e-6"
+        />
+    </inertial>
+    <visual>
+        <geometry>
+            <mesh filename="package://my_robot/meshes/hokuyo.dae"/>
+        </geometry>
+    </visual>
+  </link>
+  <joint type="fixed" name="hokuyo_joint">
+    <origin xyz="0.15 0 0.1" rpy="0 0 0"/>
+    <child link="hokuyo"/>
+    <parent link="chassis"/>
+    <axis xyz="0 1 0"/>
+  </joint>
 </robot>

Commit message: added colors

File: catkin_ws/src/my_robot/urdf/my_robot.xacro (robot description, xacro)
@@ -172,3 +172,16 @@
     <axis xyz="0 1 0"/>
   </joint>
+<!-- Test colors -->
+  <gazebo reference="left_wheel">
+    <material>Gazebo/Green</material>
+  </gazebo>
+  <gazebo reference="right_wheel">
+    <material>Gazebo/Blue</material>
+  </gazebo>
+    <gazebo reference="camera">
+    <material>Gazebo/Red</material>
+  </gazebo>
+    <gazebo reference="chassis">
+    <material>Gazebo/Gold</material>
+  </gazebo>
 </robot>

Commit message: fixed errors in world creation

File: catkin_ws/src/my_robot/urdf/my_robot.xacro (robot description, xacro)
@@ -22,5 +22,5 @@
       <origin xyz="0 0 0" rpy=" 0 0 0"/>
       <geometry>
-        <box size=".4 .2 .1"/>
+        <box size="0.4 0.2 0.1"/>
       </geometry>
     </collision>
@@ -28,5 +28,5 @@
       <origin xyz="0 0 0" rpy=" 0 0 0"/>
       <geometry>
-        <box size=".4 .2 .1"/>
+        <box size="0.4 0.2 0.1"/>
       </geometry>
     </visual>
@@ -181,8 +181,8 @@
   </gazebo>
     <gazebo reference="camera">
+    <material>Gazebo/Black</material>
+  </gazebo>
+    <gazebo reference="chassis">
     <material>Gazebo/Red</material>
   </gazebo>
-    <gazebo reference="chassis">
-    <material>Gazebo/Gold</material>
-  </gazebo>
 </robot>

Commit message: changed the model of the robot

File: catkin_ws/src/my_robot/urdf/my_robot.xacro (robot description, xacro)
@@ -22,5 +22,5 @@
       <origin xyz="0 0 0" rpy=" 0 0 0"/>
       <geometry>
-        <box size="0.4 0.2 0.1"/>
+        <box size="0.4 0.6 0.1"/>
       </geometry>
     </collision>
@@ -28,29 +28,29 @@
       <origin xyz="0 0 0" rpy=" 0 0 0"/>
       <geometry>
-        <box size="0.4 0.2 0.1"/>
+        <box size="0.4 0.6 0.1"/>
       </geometry>
     </visual>
     <collision name='back_caster_collision'>
-      <origin xyz="-0.15 0 -0.05" rpy=" 0 0 0"/>
+      <origin xyz="-0.15 0 -0.1" rpy=" 0 0 0"/>
       <geometry>
-        <sphere radius="0.0499"/>
+        <sphere radius="0.100"/>
       </geometry>
     </collision>
     <visual name='back_caster_visual'>
-      <origin xyz="-0.15 0 -0.05" rpy=" 0 0 0"/>
+      <origin xyz="-0.15 0 -0.1" rpy=" 0 0 0"/>
       <geometry>
-        <sphere radius="0.05"/>
+        <sphere radius="0.10"/>
       </geometry>
     </visual>
     <collision name='front_caster_collision'>
-      <origin xyz="0.15 0 -0.05" rpy=" 0 0 0"/>
+      <origin xyz="0.15 0 -0.1" rpy=" 0 0 0"/>
       <geometry>
-        <sphere radius="0.0499"/>
+        <sphere radius="0.100"/>
       </geometry>
     </collision>
     <visual name='front_caster_visual'>
-      <origin xyz="0.15 0 -0.05" rpy=" 0 0 0"/>
+      <origin xyz="0.15 0 -0.1" rpy=" 0 0 0"/>
       <geometry>
-        <sphere radius="0.05"/>
+        <sphere radius="0.10"/>
       </geometry>
     </visual>
@@ -60,5 +60,5 @@
         <origin xyz="0 0 0" rpy="0 1.507 1.507"/>
         <geometry>
-            <cylinder radius="0.1" length="0.05"/>
+            <cylinder radius="0.2" length="0.05"/>
         </geometry>
     </collision>
@@ -75,5 +75,5 @@
         <origin xyz="0 0 0" rpy="0 1.507 1.507"/>
         <geometry>
-            <cylinder radius="0.1" length="0.05"/>
+            <cylinder radius="0.2" length="0.05"/>
         </geometry>
     </visual>
@@ -83,5 +83,5 @@
         <origin xyz="0 0 0" rpy="0 1.507 1.507"/>
         <geometry>
-            <cylinder radius="0.1" length="0.05"/>
+            <cylinder radius="0.2" length="0.05"/>
         </geometry>
     </collision>
@@ -98,10 +98,10 @@
         <origin xyz="0 0 0" rpy="0 1.507 1.507"/>
         <geometry>
-            <cylinder radius="0.1" length="0.05"/>
+            <cylinder radius="0.2" length="0.05"/>
         </geometry>
     </visual>
   </link> -->
   <joint type="continuous" name="left_wheel_hinge">
-    <origin xyz="0 0.15 0" rpy="0 0 0"/>
+    <origin xyz="0 0.3 0" rpy="0 0 0"/>
     <child link="left_wheel"/>
     <parent link="chassis"/>
@@ -111,5 +111,5 @@
   </joint>
   <joint type="continuous" name="right_wheel_hinge">
-    <origin xyz="0 -0.15 0" rpy="0 0 0"/>
+    <origin xyz="0 -0.3 0" rpy="0 0 0"/>
     <child link="right_wheel"/>
     <parent link="chassis"/>
